File: 2_Manager_Outputs/2_Manager_Outputs.kicad_pcb (KiCad board)
At the start: 2 copper layers, 100 x 100 mm, 36 parts, among them J1 VDD 12V, J11 I2C, J2 RS232, J3 VDD 5V, J4 SPEAKER, J5 RESET, P3 SPI, SW1 Reset, U1 ATMEGA328P-AU_MIO, U4 LD1117S33TR_MIO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

Commit message: //
//
Parts:
- moved R7 64.3 mm to (88.5, 43.6), turned to 90 degrees
- moved D2 63.7 mm to (84.4, 43.6), turned to 270 degrees
- moved C33 57.5 mm to (94.2, 55.2), turned to 270 degrees
- moved R1 54.0 mm to (159.6, 102.7), turned to 180 degrees
- moved D1 53.9 mm to (159.5, 106.6), turned to 0 degrees
- moved C32 52.1 mm to (98.0, 55.2), turned to 270 degrees
- moved C4 45.8 mm to (143.1, 59.6), turned to 180 degrees
- moved C5 41.5 mm to (143.1, 57.4), turned to 180 degrees
- moved J3 32.7 mm to (164.2, 115.2), turned to 180 degrees
- moved R2 30.1 mm to (134.9, 55.8), turned to 90 degrees
- moved C8 24.4 mm to (165.8, 102.6), turned to 180 degrees
- moved D3 22.2 mm to (132.4, 55.7), turned to 270 degrees
- moved C9 19.1 mm to (165.7, 106.5), turned to 180 degrees

Commit message: //
//
Parts:
- moved J4 45.1 mm to (100.6, 24.5)
- moved C2 11.9 mm to (120.4, 53.5)
- moved D3 11.9 mm to (127.8, 44.7)
- moved U4 11.9 mm to (121.7, 47.2)
- moved C1 11.9 mm to (116.6, 48.5)
- moved JP2 11.9 mm to (113.0, 49.8)
- moved R2 11.9 mm to (130.3, 44.8)
- moved JP3 11.9 mm to (125.3, 54.2)
- moved C7 1.70 mm to (139.2, 63.5)
- moved C6 1.15 mm to (139.2, 61.3)
- moved C4 0.81 mm to (142.5, 59.0)
- moved C5 0.80 mm to (142.5, 56.8)
- moved JP1 0.12 mm to (160.2, 59.7)
Changed lines of the file:
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@@
     (links 131)
     (no_connects 131)
-    (area 79.34044 20.75592 180.78408 122.075001)
+    (area 79.924999 21.924999 180.075001 122.075001)
     (thickness 1.6)
     (drawings 4)
@@
   )
   (module TO_SOT_Packages_SMD:SOT-223 (layer F.Cu)
-    (at 126.27 58.24)
+    (at 121.65 47.23)
     (descr "module CMS SOT223 4 pins")
     (tags "CMS SOT")
@@
   )
   (module Resistors_SMD:R_0805_HandSoldering (layer F.Cu)
-    (at 121.23 59.47 270)
+    (at 116.61 48.46 270)
     (descr "Resistor SMD 0805, hand soldering")
     (tags "resistor 0805")
@@
   )
   (module Resistors_SMD:R_0805_HandSoldering (layer F.Cu)
-    (at 124.98 64.54 180)
+    (at 120.36 53.53 180)
     (descr "Resistor SMD 0805, hand soldering")
     (tags "resistor 0805")
@@
   )
   (module Resistors_SMD:R_0805_HandSoldering (layer F.Cu)
-    (at 143.09 59.56 180)
+    (at 142.49 59.02 180)
     (descr "Resistor SMD 0805, hand soldering")
     (tags "resistor 0805")
@@
   )
   (module Resistors_SMD:R_0805_HandSoldering (layer F.Cu)
-    (at 143.1 57.37 180)
+    (at 142.5 56.84 180)
     (descr "Resistor SMD 0805, hand soldering")
     (tags "resistor 0805")
@@
   )
   (module Socket_Strips:Socket_Strip_Straight_1x02 (layer F.Cu)
-    (at 117.59 60.82 90)
+    (at 112.97 49.81 90)
     (descr "Through hole socket strip")
     (tags "socket strip")
@@
   )
   (module Socket_Strips:Socket_Strip_Straight_1x02 (layer F.Cu)
-    (at 129.89 65.21)
+    (at 125.27 54.2)
     (descr "Through hole socket strip")
     (tags "socket strip")
@@
   )
   (module Resistors_SMD:R_0805_HandSoldering (layer F.Cu)
-    (at 138.03 61.12 180)
+    (at 139.17 61.27 180)
     (descr "Resistor SMD 0805, hand soldering")
     (tags "resistor 0805")
@@
   )
   (module Resistors_SMD:R_0805_HandSoldering (layer F.Cu)
-    (at 138.19 64.93 180)
+    (at 139.17 63.54 180)
     (descr "Resistor SMD 0805, hand soldering")
     (tags "resistor 0805")
@@
   )
   (module Resistors_SMD:R_0805_HandSoldering (layer F.Cu)
-    (at 132.44 55.74 270)
+    (at 127.82 44.73 270)
     (descr "Resistor SMD 0805, hand soldering")
     (tags "resistor 0805")
@@
   )
   (module Resistors_SMD:R_0805_HandSoldering (layer F.Cu)
-    (at 134.91 55.78 90)
+    (at 130.29 44.77 90)
     (descr "Resistor SMD 0805, hand soldering")
     (tags "resistor 0805")
@@
   )
   (module Socket_Strips:Socket_Strip_Straight_1x02 (layer F.Cu)
-    (at 140.59 45.42 180)
+    (at 100.63 24.54 180)
     (descr "Through hole socket strip")
     (tags "socket strip")
@@
     (tags "resistor 0805")
     (attr smd)
-    (fp_text reference C10 (at 0 -2.1 180) (layer F.SilkS)
+    (fp_text reference C10 (at -4.07 -0.07 180) (layer F.SilkS)
       (effects (font (size 1 1) (thickness 0.15)))
     )
@@
   )
   (module Resistors_SMD:R_0805_HandSoldering (layer F.Cu)
-    (at 160.35 59.71 180)
+    (at 160.23 59.74 180)
     (descr "Resistor SMD 0805, hand soldering")
     (tags "resistor 0805")

Commit message: //
//
Parts:
- moved R3 14.2 mm to (151.2, 50.6), turned to 270 degrees
- moved SW1 2.40 mm to (149.6, 40.1), turned to 90 degrees
- moved C5 0.99 mm to (141.5, 56.9)
- moved C4 0.96 mm to (141.5, 59.0)
- moved C7 0.31 mm to (139.4, 63.4)
- moved Y1 0.28 mm to (143.6, 62.3)
- moved C6 0.27 mm to (139.4, 61.2)
Connections:
- J11 pad 1: /SDA -> /SCL
- J11 pad 2: /SCL -> /SDA
Routing:
- net /+5V: track 0.00 -> 179.1 mm
- net /GND: track 0.00 -> 87.9 mm, vias 0 -> 15
- net /ACTIVAR_RETORNO: track 0.00 -> 72.2 mm
- net /SPEAKER: track 0.00 -> 65.2 mm
- net /ACTIVAR_CORTE: track 0.00 -> 50.8 mm
- net /VDD: track 0.00 -> 43.6 mm
- net /SCL: track 0.00 -> 41.5 mm
- net /MEDIR_Z_L_COMUN: track 0.00 -> 39.6 mm
- net /SDA: track 0.00 -> 37.8 mm
- net /+12V: track 0.00 -> 37.7 mm
- net /SD_LAPIZ_COAG: track 0.00 -> 37.7 mm
- net /Tx: track 0.00 -> 35.9 mm
- net /SD_LAPIZ_CORTE: track 0.00 -> 35.7 mm
- net /Rx: track 0.00 -> 35.2 mm
- net /SD_LAPIZ_COM: track 0.00 -> 33.8 mm
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- added copper zone on B.Cu, net /GND
Other:
- net class Default: clearance 0.2 -> 0.18; trace_width 0.25 -> 0.2
- rule trace_clearance: 0.2 -> 0.18
- rule trace_min: 0.2 -> 0.1524
- rule via_min_size: 0.4 -> 0.5
