File: 2_Manager_Outputs/2_Manager_Outputs.kicad_pcb (KiCad board)
At the start: 2 copper layers, 100 x 100 mm, 36 parts, among them J1 VDD 12V, J11 I2C, J2 RS232, J3 VDD 5V, J4 SPEAKER, J5 RESET, P3 SPI, SW1 Reset, U1 ATMEGA328P-AU_MIO, U4 LD1117S33TR_MIO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

Commit message: //
//
Parts:
- moved U4 7.52 mm to (124.3, 54.3), turned to 270 degrees
- moved JP3 6.46 mm to (131.7, 54.1)
- moved C1 6.26 mm to (118.4, 54.5), turned to 90 degrees
- moved D3 6.19 mm to (133.6, 46.9)
- moved R2 6.19 mm to (136.1, 47.0)
- moved JP2 6.04 mm to (108.7, 54.0), turned to 0 degrees
- moved C2 4.49 mm to (122.5, 49.6)
Routing:
- net /ACTIVAR_RETORNO: track 72.2 -> 143.3 mm, vias 0 -> 1
- net /GND: track 87.9 -> 145.9 mm, vias 15 -> 20
- net /ACTIVAR_COAG: track 10.2 -> 65.9 mm, vias 0 -> 1
- net /VDD: track 43.6 -> 83.8 mm, vias 0 -> 3
- net /+12V: track 37.7 -> 21.0 mm
- net Net-(C1-Pad1): track 14.0 -> 2.95 mm
- net Net-(C2-Pad1): track 6.86 -> 15.8 mm
- added copper zone on F.Cu, net /+12V
- added copper zone on F.Cu, net /GND
- added copper zone on F.Cu, net /VDD
- added copper zone on F.Cu, net Net-(C1-Pad1)
- added copper zone on F.Cu, net Net-(C2-Pad1)
