File: 4_Wave_Generator/2_Manager_Outputs.sch (KiCad schematic (older format))
At the start: 42 parts, among them J1 Jumper, J10 SPI_AD9833, J11 I2C, J15 Jumper, J2 RS232, J3 Jumper, J4 Jumper, J5 Jumper, J6 Jumper, J7 Jumper, J8 Jumper, J9 Jumper, P1 MCLK_EXTERNAL, P2 CONN_01X04, P3 SPI_ATMEGA, P4 CONN_01X04, U1 ATMEGA328P-AU_MIO, U2 AD8421, U3 AD9833, U4 LD1117S33TR_MIO, U9 ADG819

Commit message: //
//
Parts:
- removed J10: SPI_AD9833, Pin_Headers:Pin_Header_Straight_1x03, symbol CONN_01X03
- removed J11: I2C, Pin_Headers:Pin_Header_Straight_1x02, symbol CONN_01X02
- removed J2: RS232, Pin_Headers:Pin_Header_Straight_1x03, symbol CONN_01X03
- removed P3: SPI_ATMEGA, Socket_Strips:Socket_Strip_Straight_1x04, symbol CONN_01X04
- removed U4: LD1117S33TR_MIO, TO_SOT_Packages_SMD:SOT-223, symbol LD1117S33TR_MIO
- added C? (x2): 0.1uF, Capacitors_SMD:C_0805_HandSoldering, symbol 0.1uF
- added C? (x2): 10uF, Capacitors_SMD:C_0805_HandSoldering, symbol 10uF
- added C? (x5): 0.1uF, Resistors_SMD:R_0805_HandSoldering, symbol 0.1uF
- added C?: 10uF, Resistors_SMD:R_0805_HandSoldering, symbol 10uF
- added C? (x2): 8pF, Resistors_SMD:R_0805_HandSoldering, symbol 20pF
- added D?: 12V, Resistors_SMD:R_0805_HandSoldering, symbol Led_0805
- added D?: 5V, Resistors_SMD:R_0805_HandSoldering, symbol Led_0805
- added D?: VDD, Resistors_SMD:R_0805_HandSoldering, symbol Led_0805
- added J?: RS232, Foot_Prints_Manager_Outputs:RS232, symbol CONN_01X03
- added J?: I2C, Foot_Prints_Manager_Outputs:I2C_2X4, symbol CONN_01X02
- added J?: VDD 12V, Foot_Prints_Manager_Outputs:SUPPLY_12V, symbol CONN_01X02
- added J?: VDD 5V, Foot_Prints_Manager_Outputs:SUPPLY_5V, symbol CONN_01X02
- added J?: SPEAKER, Socket_Strips:Socket_Strip_Straight_1x02, symbol CONN_01X02
- added J?: RESET, Foot_Prints_Manager_Outputs:RESET_CONNECTOR, symbol CONN_01X02
- added JP?: J_VDD, Socket_Strips:Socket_Strip_Straight_1x02, symbol Jumper_NC_Small
- added JP?: J_+12V, Socket_Strips:Socket_Strip_Straight_1x02, symbol Jumper_NC_Small
- added P?: SPI, Foot_Prints_Manager_Outputs:SPI_CONNECTOR, symbol CONN_01X04
- added R? (x3): 1K, Resistors_SMD:R_0805_HandSoldering, symbol 1K
- added R?: 10K, Resistors_SMD:R_0805_HandSoldering, symbol 10K
- added SW?: Reset, Huellas:KPT_1187B, symbol SW_Push
- added U?: LD1117S33TR_MIO, TO_SOT_Packages_SMD:SOT-223, symbol LD1117S33TR_MIO
- added Y?: Crystal, Huellas:Crystal_SMD_XRCHA_Murata_Serie_W2,5mm_L2,0mm, symbol Crystal_Small
Connections:
- net labels added: +5V, DTR, SPEAKER
- wire segments 142 -> 199
- no-connect marks 2 -> 4
Other:
- note added: "CRYSTAL \nOSCILLATOR"
- note added: "DECUPLING CAPACITORS"
- note added: "DIGITAL BUSES AND CONNECTORS"
- note added: "INDICATORS LEDS"
- note added: "RESET"
- note removed: "PINES PROGRAMACIÓN"
- moved on the sheet: C1, C12, C13, C14, C3, C31, C32, C33, C4, C6, C7, C8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

Commit message: //
//
Parts:
- removed SW?: Reset, Huellas:KPT_1187B, symbol SW_Push
- added C?: 1nF, Capacitors_SMD:C_0805_HandSoldering, symbol 1nF
- added C?: 1.5nF, Capacitors_SMD:C_0805_HandSoldering, symbol 1.5nF
- added C? (x4): 0.1uF, Capacitors_SMD:C_0805_HandSoldering, symbol 0.1uF
- added C? (x2): 0.33uF, Capacitors_SMD:C_0805_HandSoldering, symbol 0.33uF
- added C? (x2): 22pF, Capacitors_SMD:C_0805_HandSoldering, symbol 22pF
- added C?: 10nF, Capacitors_SMD:C_0805_HandSoldering, symbol 10nF
- added D?: LED, LEDs:LED_0805, symbol LED
- added JP?: PASO_A/D, Pin_Headers:Pin_Header_Straight_1x02_Pitch2.54mm, symbol PASO_A/D
- added P?: ECG INPUTS, Huellas:Pin_Header_Straight_1x03_Pitch2.54mm, symbol CONN_01X03-RESCUE-proyectos
- added P?: PIC_PROGRAMER, Pin_Headers:Pin_Header_Angled_1x05_Pitch2.54mm, symbol CONN_01X05
- added P?: AD8232_CONTROL, Pin_Headers:Pin_Header_Straight_1x03_Pitch2.54mm, symbol CONN_01X03-RESCUE-proyectos
- added P?: PIC_OUTPUTS, Pin_Headers:Pin_Header_Straight_1x03_Pitch2.54mm, symbol CONN_01X03
- added R? (x6): 10M, Resistors_SMD:R_0805_HandSoldering, symbol 10M
- added R? (x2): 180K, Resistors_SMD:R_0805_HandSoldering, symbol 180K
- added R?: 360K, Resistors_SMD:R_0805_HandSoldering, symbol 360K
- added R? (x3): 1M, Resistors_SMD:R_0805_HandSoldering, symbol 1M
- added R?: 100K, Resistors_SMD:R_0805_HandSoldering, symbol 100K
- added R?: 1.4M, Resistors_SMD:R_0805_HandSoldering, symbol 1.4M
- added R? (x2): 1K, Resistors_SMD:R_0805_HandSoldering, symbol 1K
- added R? (x2): 10K, Resistors_SMD:R_0805_HandSoldering, symbol 10K
- added SW?: SW_Push, symbol SW_Push
- added SW?: RESET_PIC, symbol SW_Push
- added U?: PIC16F688, Housings_SOIC:SOIC-14_3.9x8.7mm_Pitch1.27mm, symbol PIC16F688
- added U?: AD8232_A, Huellas:AD8232_ECG, symbol AD8232_A
- added Y?: Crystal_8MHz, Crystals:Crystal_SMD_Abracon_ABM3-2pin_5.0x3.2mm_HandSoldering, symbol Crystal_8MHz
Connections:
- net labels added: +vs, ADC, IAOUT, ICSPCLK, ICSPDAT, LA, LOD+, LOD-, MCLR/Vpp, OPAMP+, OPAMP-, OUT_ANALOG, O_DIG1, O_DIG2, RA, REFIN, REFOUT, RL, RLD, RLDFB, SDN, SDN_OFF, SW, VCC
- wire segments 199 -> 299
Other:
- note added: "ACTUALIZAR CON TODAS LAS SALIDAS"
- note added: "BLOQUE DE ADQUISICION DE ECG"
- note added: "CONECCION ENTRE A/D\n"
- note added: "CONECTORES DE SALIDA/ENTRADA"
- note added: "CONVERTIDOR ANALOGICO A DIGITAL\n"
- note added: "ENTRADA DE CONTROL\n DE APAGADO DEL ECG"
- note added: "IND. ECG\n"
- note added: "INDICADORES LED\n"
- note added: "SI, SE PUEDE ENVIAR AL MICRO"
- moved on the sheet: C1, C12, C13, C14, C3, C31, C32, C33, C4, C6, C7, C8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
