File: 4_Wave_Generator/4_Wave_Generator.kicad_pcb (KiCad board)
At the start: 2 copper layers, 103 parts, among them J1 RS232, J10 Jumper, J11 Jumper, J12 Jumper, J13 Jumper, J14 Jumper, J15 Jumper, J2 I2C, J3 SPEAKER, J4 RESET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

Commit message: //
//
Parts:
- moved P6 21.6 mm to (143.9, 50.2)
Changed lines of the file:
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@@
   )
   (module Pin_Headers:Pin_Header_Angled_1x04_Pitch2.54mm (layer F.Cu)
-    (at 160.19 35.96)
+    (at 143.87 50.18)
     (descr "Through hole angled pin header, 1x04, 2.54mm pitch, 6mm pin length, single row")
     (tags "Through hole angled pin header THT 1x04 2.54mm single row")
